Commit message: Add a prefix for Panda arm links and joints

File: doc/examples/dual_arms/dual_arm_panda_moveit_config/config/panda.urdf.xacro (robot description, xacro)
@@ -2,10 +2,22 @@
 <robot xmlns:xacro="http://www.ros.org/wiki/xacro" name="panda">
     <xacro:arg name="initial_positions_file" default="initial_positions.yaml" />
-    <!-- Import panda urdf file -->
-    <xacro:include filename="$(find moveit_resources_panda_description)/urdf/panda.urdf" />
-    <!-- Import panda ros2_control description -->
+    <!-- Xacro imports -->
+    <xacro:include filename="panda_arm_macro.xacro" />
     <xacro:include filename="panda.ros2_control.xacro" />
     <xacro:include filename="panda_hand.ros2_control.xacro" />
     <xacro:panda_ros2_control name="PandaFakeSystem" initial_positions_file="$(arg initial_positions_file)"/>
     <xacro:panda_hand_ros2_control name="PandaHandFakeSystem"/>
+    <link name="world"/>
+    <!-- Left arm -->
+    <xacro:panda_arm
+        prefix="left_"
+        parent="world">
+        <origin xyz="0 -1.5 0" rpy="0 0 0" />
+    </xacro:panda_arm>
+    <!-- Right arm -->
+    <xacro:panda_arm
+        prefix="right_"
+        parent="world">
+        <origin xyz="0 1.5 0" rpy="0 0 0" />
+    </xacro:panda_arm>
 </robot>
