Commit message: Update initial joint positions

File: doc/examples/dual_arms/dual_arm_panda_moveit_config/config/panda.ros2_control.xacro (robot description, xacro)
@@ -1,5 +1,5 @@
 <?xml version="1.0"?>
 <robot xmlns:xacro="http://www.ros.org/wiki/xacro">
-    <xacro:macro name="panda_ros2_control" params="name initial_positions_file">
+    <xacro:macro name="panda_ros2_control" params="name initial_positions_file prefix">
         <xacro:property name="initial_positions" value="${load_yaml(initial_positions_file)['initial_positions']}"/>
         <ros2_control name="${name}" type="system">
@@ -7,5 +7,5 @@
                 <plugin>fake_components/GenericSystem</plugin>
             </hardware>
-            <joint name="panda_joint1">
+            <joint name="${prefix}panda_joint1">
                 <command_interface name="position"/>
                 <state_interface name="position">
@@ -14,5 +14,5 @@
                 <state_interface name="velocity"/>
             </joint>
-            <joint name="panda_joint2">
+            <joint name="${prefix}panda_joint2">
                 <command_interface name="position"/>
                 <state_interface name="position">
@@ -21,5 +21,5 @@
                 <state_interface name="velocity"/>
             </joint>
-            <joint name="panda_joint3">
+            <joint name="${prefix}panda_joint3">
                 <command_interface name="position"/>
                 <state_interface name="position">
@@ -28,5 +28,5 @@
                 <state_interface name="velocity"/>
             </joint>
-            <joint name="panda_joint4">
+            <joint name="${prefix}panda_joint4">
                 <command_interface name="position"/>
                 <state_interface name="position">
@@ -35,5 +35,5 @@
                 <state_interface name="velocity"/>
             </joint>
-            <joint name="panda_joint5">
+            <joint name="${prefix}panda_joint5">
                 <command_interface name="position"/>
                 <state_interface name="position">
@@ -42,5 +42,5 @@
                 <state_interface name="velocity"/>
             </joint>
-            <joint name="panda_joint6">
+            <joint name="${prefix}panda_joint6">
                 <command_interface name="position"/>
                 <state_interface name="position">
@@ -49,5 +49,5 @@
                 <state_interface name="velocity"/>
             </joint>
-            <joint name="panda_joint7">
+            <joint name="${prefix}panda_joint7">
                 <command_interface name="position"/>
                 <state_interface name="position">

File: doc/examples/dual_arms/dual_arm_panda_moveit_config/config/panda.urdf.xacro (robot description, xacro)
@@ -1,22 +1,28 @@
 <?xml version="1.0"?>
 <robot xmlns:xacro="http://www.ros.org/wiki/xacro" name="panda">
-    <xacro:arg name="initial_positions_file" default="initial_positions.yaml" />
+    <xacro:arg name="left_initial_positions_file"
+            default="$(find dual_arm_panda_moveit_config)/config/left_initial_positions.yaml"/>
+    <xacro:arg name="right_initial_positions_file"
+            default="$(find dual_arm_panda_moveit_config)/config/right_initial_positions.yaml"/>
     <!-- Xacro imports -->
     <xacro:include filename="panda_arm_macro.xacro" />
     <xacro:include filename="panda.ros2_control.xacro" />
     <xacro:include filename="panda_hand.ros2_control.xacro" />
-    <xacro:panda_ros2_control name="PandaFakeSystem" initial_positions_file="$(arg initial_positions_file)"/>
-    <xacro:panda_hand_ros2_control name="PandaHandFakeSystem"/>
+    <!-- Root link -->
     <link name="world"/>
     <!-- Left arm -->
     <xacro:panda_arm
+        name="left_panda"
         prefix="left_"
-        parent="world">
+        parent="world"
+        initial_positions_file="$(arg left_initial_positions_file)">
         <origin xyz="0 -1.5 0" rpy="0 0 0" />
     </xacro:panda_arm>
     <!-- Right arm -->
     <xacro:panda_arm
+        name="right_panda"
         prefix="right_"
-        parent="world">
+        parent="world"
+        initial_positions_file="$(arg right_initial_positions_file)">
         <origin xyz="0 1.5 0" rpy="0 0 0" />
     </xacro:panda_arm>

File: doc/examples/dual_arms/dual_arm_panda_moveit_config/config/panda_arm_macro.xacro (robot description, xacro)
@@ -1,5 +1,8 @@
 <?xml version="1.0" ?>
 <robot xmlns:xacro="http://www.ros.org/wiki/xacro">
-    <xacro:macro name="panda_arm" params="prefix parent *origin" >
+    <xacro:macro name="panda_arm" params="name prefix parent *origin initial_positions_file" >
+        <!-- ros2_control -->
+        <xacro:include filename="$(find dual_arm_panda_moveit_config)/config/panda.ros2_control.xacro" />
+        <xacro:panda_ros2_control name="${name}" initial_positions_file="${initial_positions_file}" prefix="${prefix}"/>
         <!-- base_joint fixes base_link to the environment -->
         <joint name="${prefix}base_joint" type="fixed">

Commit message: MoveIt planning works!

File: doc/examples/dual_arms/dual_arm_panda_moveit_config/config/panda.ros2_control.xacro (robot description, xacro)
@@ -1,7 +1,7 @@
 <?xml version="1.0"?>
 <robot xmlns:xacro="http://www.ros.org/wiki/xacro">
-    <xacro:macro name="panda_ros2_control" params="name initial_positions_file prefix">
+    <xacro:macro name="panda_arm_ros2_control" params="name initial_positions_file prefix">
         <xacro:property name="initial_positions" value="${load_yaml(initial_positions_file)['initial_positions']}"/>
-        <ros2_control name="${name}" type="system">
+        <ros2_control name="${prefix}${name}" type="system">
             <hardware>
                 <plugin>fake_components/GenericSystem</plugin>

File: doc/examples/dual_arms/dual_arm_panda_moveit_config/config/panda.urdf.xacro (robot description, xacro)
@@ -5,10 +5,8 @@
     <xacro:arg name="right_initial_positions_file"
             default="$(find dual_arm_panda_moveit_config)/config/right_initial_positions.yaml"/>
+    <!-- Root link -->
+    <link name="world"/>
     <!-- Xacro imports -->
     <xacro:include filename="panda_arm_macro.xacro" />
-    <xacro:include filename="panda.ros2_control.xacro" />
-    <xacro:include filename="panda_hand.ros2_control.xacro" />
-    <!-- Root link -->
-    <link name="world"/>
     <!-- Left arm -->
     <xacro:panda_arm

File: doc/examples/dual_arms/dual_arm_panda_moveit_config/config/panda_arm_macro.xacro (robot description, xacro)
@@ -4,5 +4,7 @@
         <!-- ros2_control -->
         <xacro:include filename="$(find dual_arm_panda_moveit_config)/config/panda.ros2_control.xacro" />
-        <xacro:panda_ros2_control name="${name}" initial_positions_file="${initial_positions_file}" prefix="${prefix}"/>
+        <xacro:panda_arm_ros2_control name="${name}" initial_positions_file="${initial_positions_file}" prefix="${prefix}"/>
+        <xacro:include filename="panda_hand.ros2_control.xacro" />
+        <xacro:panda_hand_ros2_control name="${name}" prefix="${prefix}"/>
         <!-- base_joint fixes base_link to the environment -->
         <joint name="${prefix}base_joint" type="fixed">
@@ -226,5 +228,5 @@
             <axis xyz="0 -1 0" />
             <limit effort="20" lower="0.0" upper="0.04" velocity="0.2" />
-            <mimic joint="panda_finger_joint1" />
+            <mimic joint="${prefix}panda_finger_joint1" />
         </joint>
     </xacro:macro>

File: doc/examples/dual_arms/dual_arm_panda_moveit_config/config/panda_hand.ros2_control.xacro (robot description, xacro)
@@ -1,10 +1,10 @@
 <?xml version="1.0"?>
 <robot xmlns:xacro="http://www.ros.org/wiki/xacro">
-    <xacro:macro name="panda_hand_ros2_control" params="name">
+    <xacro:macro name="panda_hand_ros2_control" params="name prefix">
         <ros2_control name="${name}" type="system">
             <hardware>
                 <plugin>fake_components/GenericSystem</plugin>
             </hardware>
-            <joint name="panda_finger_joint1">
+            <joint name="${prefix}panda_finger_joint1">
                 <command_interface name="position" />
                 <state_interface name="position">
@@ -13,6 +13,6 @@
                 <state_interface name="velocity"/>
             </joint>
-            <joint name="panda_finger_joint2">
-                <param name="mimic">panda_finger_joint1</param>
+            <joint name="${prefix}panda_finger_joint2">
+                <param name="mimic">${prefix}panda_finger_joint1</param>
                 <param name="multiplier">1</param>
                 <command_interface name="position" />
